File: pwr_supply/pwr_supply.sch (KiCad schematic (older format))
At the start: 15 parts, among them J1 Barrel_Jack_Switch, J2 Conn_02x02_Odd_Even, J3 Conn_02x02_Odd_Even, SW1 SW_DPDT_x2, U1 LM7805_TO220

Commit message: pwr_supply
Parts:
- C1: footprint (none) -> Capacitor_THT:CP_Radial_D10.0mm_P5.00mm
- C2: footprint (none) -> Capacitor_THT:CP_Radial_D6.3mm_P2.50mm
- D5, D6: footprint (none) -> LED_THT:LED_D5.0mm
- J1: footprint (none) -> Connector_BarrelJack:BarrelJack_CUI_PJ-102AH_Horizontal
- J2, J3: footprint (none) -> Connector_PinHeader_2.54mm:PinHeader_2x02_P2.54mm_Vertical
- R1, R2: footprint (none) -> Resistor_THT:R_Axial_DIN0207_L6.3mm_D2.5mm_P7.62mm_Horizontal
- SW1: footprint (none) -> dk_st_fp:Switch_Slide_11.6x4mm_EG1218
Changed lines of the file:
@@
 F 0 "J1" H 2557 4067 50  0000 C CNN
 F 1 "Barrel_Jack_Switch" H 2557 3976 50  0000 C CNN
-F 2 "" H 2550 3710 50  0001 C CNN
+F 2 "Connector_BarrelJack:BarrelJack_CUI_PJ-102AH_Horizontal" H 2550 3710 50  0001 C CNN
 F 3 "~" H 2550 3710 50  0001 C CNN
 	1    2500 3750
@@
 F 0 "C1" H 4568 3696 50  0000 L CNN
 F 1 "CP" H 4568 3605 50  0000 L CNN
-F 2 "" H 4488 3500 50  0001 C CNN
+F 2 "Capacitor_THT:CP_Radial_D10.0mm_P5.00mm" H 4488 3500 50  0001 C CNN
 F 3 "~" H 4450 3650 50  0001 C CNN
 	1    4450 3650
@@
 F 0 "C2" H 5818 3696 50  0000 L CNN
 F 1 "CP" H 5818 3605 50  0000 L CNN
-F 2 "" H 5738 3500 50  0001 C CNN
+F 2 "Capacitor_THT:CP_Radial_D6.3mm_P2.50mm" H 5738 3500 50  0001 C CNN
 F 3 "~" H 5700 3650 50  0001 C CNN
 	1    5700 3650
@@
 F 0 "R1" H 6170 3696 50  0000 L CNN
 F 1 "R" H 6170 3605 50  0000 L CNN
-F 2 "" V 6030 3650 50  0001 C CNN
+F 2 "Resistor_THT:R_Axial_DIN0207_L6.3mm_D2.5mm_P7.62mm_Horizontal" V 6030 3650 50  0001 C CNN
 F 3 "~" H 6100 3650 50  0001 C CNN
 	1    6100 3650
@@
 F 0 "D5" V 6139 3932 50  0000 R CNN
 F 1 "LED" V 6048 3932 50  0000 R CNN
-F 2 "" H 6100 4050 50  0001 C CNN
+F 2 "LED_THT:LED_D5.0mm" H 6100 4050 50  0001 C CNN
 F 3 "~" H 6100 4050 50  0001 C CNN
 	1    6100 4050
@@
 F 0 "SW1" H 6450 3485 50  0000 C CNN
 F 1 "SW_DPDT_x2" H 6450 3394 50  0000 C CNN
-F 2 "" H 6450 3200 50  0001 C CNN
+F 2 "dk_st_fp:Switch_Slide_11.6x4mm_EG1218" H 6450 3200 50  0001 C CNN
 F 3 "~" H 6450 3200 50  0001 C CNN
 	1    6450 3200
@@
 F 0 "R2" H 6870 3696 50  0000 L CNN
 F 1 "R" H 6870 3605 50  0000 L CNN
-F 2 "" V 6730 3650 50  0001 C CNN
+F 2 "Resistor_THT:R_Axial_DIN0207_L6.3mm_D2.5mm_P7.62mm_Horizontal" V 6730 3650 50  0001 C CNN
 F 3 "~" H 6800 3650 50  0001 C CNN
 	1    6800 3650
@@
 F 0 "D6" V 6839 3932 50  0000 R CNN
 F 1 "LED" V 6748 3932 50  0000 R CNN
-F 2 "" H 6800 4050 50  0001 C CNN
+F 2 "LED_THT:LED_D5.0mm" H 6800 4050 50  0001 C CNN
 F 3 "~" H 6800 4050 50  0001 C CNN
 	1    6800 4050
@@
 F 0 "J2" H 7700 3567 50  0000 C CNN
 F 1 "Conn_02x02_Odd_Even" H 7700 3476 50  0000 C CNN
-F 2 "" H 7650 3350 50  0001 C CNN
+F 2 "Connector_PinHeader_2.54mm:PinHeader_2x02_P2.54mm_Vertical" H 7650 3350 50  0001 C CNN
 F 3 "~" H 7650 3350 50  0001 C CNN
 	1    7650 3350
@@
 F 0 "J3" H 7700 4167 50  0000 C CNN
 F 1 "Conn_02x02_Odd_Even" H 7700 4076 50  0000 C CNN
-F 2 "" H 7650 3950 50  0001 C CNN
+F 2 "Connector_PinHeader_2.54mm:PinHeader_2x02_P2.54mm_Vertical" H 7650 3950 50  0001 C CNN
 F 3 "~" H 7650 3950 50  0001 C CNN
 	1    7650 3950
