File: pwr_supply/pwr_supply.kicad_pcb (KiCad board)
At the start: 2 copper layers, 30.1 x 52.1 mm, 15 parts, among them J1 Barrel_Jack_Switch, J2 Conn_02x02_Odd_Even, J3 Conn_02x02_Odd_Even, SW1 SW_DPDT_x2, U1 LM7805_TO220

Commit message: pcb
Parts:
- moved C2 63.3 mm to (137.0, 70.5)
- moved U1 62.0 mm to (126.1, 80.5)
- moved D6 57.9 mm to (141.8, 79.4)
- moved C1 56.8 mm to (126.4, 70.5)
- moved R2 51.7 mm to (137.2, 77.1), turned to 270 degrees
- moved R1 48.7 mm to (141.7, 104.6), turned to 270 degrees
- moved D2 48.5 mm to (124.8, 87.8)
- moved D4 48.4 mm to (124.8, 91.3)
- moved D5 44.8 mm to (141.8, 98.6)
- moved J1 38.5 mm to (137.4, 108.8), turned to 270 degrees
- moved D3 35.6 mm to (124.8, 98.4)
- moved D1 35.5 mm to (124.8, 94.9)
- moved SW1 33.4 mm to (143.1, 91.4), turned to 90 degrees
- moved J3 0.28 mm to (148.7, 110.6)
- moved J2 0.25 mm to (148.7, 65.6)

Commit message: finish part 1
Parts:
- added G***: LOGO, logo:logo, B.Cu at (130.3, 70.7)
- J2, J3: moved to B.Cu
- moved R1 6.12 mm to (142.2, 110.7), turned to 90 degrees
- moved R2 3.69 mm to (136.9, 73.4)
- moved D3 3.29 mm to (126.4, 101.3)
- moved J3 2.54 mm to (151.3, 110.6), turned to 180 degrees
- moved D1 2.34 mm to (126.4, 96.6)
- moved J2 2.16 mm to (150.9, 65.7), turned to 180 degrees
- moved C2 1.91 mm to (137.2, 68.6)
- moved D4 1.65 mm to (126.4, 91.9)
- moved D2 1.61 mm to (126.4, 87.2)
Routing:
- net /GND: track 0.00 -> 89.4 mm
- net /Vout2: track 0.00 -> 66.2 mm
- net /Vout1: track 0.00 -> 53.6 mm
- net /Vin: track 0.00 -> 32.1 mm
- net Net-(D1-Pad2): track 0.00 -> 29.1 mm
- net Net-(D3-Pad2): track 0.00 -> 23.7 mm
- net Net-(D6-Pad2): track 0.00 -> 10.7 mm
- net Net-(D5-Pad2): track 0.00 -> 5.45 mm
- added copper zone on B.Cu, net /GND
Other:
- board text added: "470uF"
- board text added: "47uF"
- board text added: "560R"
- board text added: "5V"
- board text added: "GND"
